Commit message: Added lower legs to mini_cheetah_mesh.urdf

File: src/quadruped_drake/models/mini_cheetah/mini_cheetah_mesh.urdf (robot description, URDF)
Before this commit: robot mini_cheetah, 17 links, 16 joints
Links:
- link shank_fl: geometry visual mesh filename=meshes/mini_lower_link.obj
- link shank_fr: geometry visual mesh filename=meshes/mini_lower_link.obj
- link shank_hl: geometry visual mesh filename=meshes/mini_lower_link.obj
- link shank_hr: geometry visual mesh filename=meshes/mini_lower_link.obj
